File: connectors.kicad_sch (KiCad schematic)
At the start: 4 parts

Commit message: Done
Parts:
- gave numbers to parts that had none: 4
Changed lines of the file:
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@@
   (symbol (lib_id "Connector:Conn_01x04_Male") (at 173.2788 68.58 0) (unit 1)
     (in_bom yes) (on_board yes) (fields_autoplaced)
-    (property "Reference" "J?" (id 0) (at 173.9138 60.4012 0))
+    (property "Reference" "J3" (id 0) (at 173.9138 60.4012 0))
     (property "Value" "Conn_01x04_Male" (id 1) (at 173.9138 62.9412 0))
     (property "Footprint" "Connector_PinHeader_2.54mm:PinHeader_1x04_P2.54mm_Vertical" (id 2) (at 173.2788 68.58 0)
@@
   (symbol (lib_id "Connector_Generic:Conn_02x03_Odd_Even") (at 175.6664 111.2012 0) (unit 1)
     (in_bom yes) (on_board yes) (fields_autoplaced)
-    (property "Reference" "J?" (id 0) (at 176.9364 102.0826 0))
+    (property "Reference" "J4" (id 0) (at 176.9364 102.0826 0))
     (property "Value" "Conn_02x03_Odd_Even" (id 1) (at 176.9364 104.6226 0))
     (property "Footprint" "Connector_PinHeader_2.54mm:PinHeader_2x03_P2.54mm_Vertical" (id 2) (at 175.6664 111.2012 0)
@@
   (symbol (lib_id "Connector:Conn_01x09_Male") (at 114.6048 114.6048 0) (unit 1)
     (in_bom yes) (on_board yes) (fields_autoplaced)
-    (property "Reference" "J?" (id 0) (at 115.2398 99.4664 0))
+    (property "Reference" "J2" (id 0) (at 115.2398 99.4664 0))
     (property "Value" "Conn_01x09_Male" (id 1) (at 115.2398 102.0064 0))
     (property "Footprint" "Connector_PinHeader_2.54mm:PinHeader_1x09_P2.54mm_Vertical" (id 2) (at 114.6048 114.6048 0)
@@
   (symbol (lib_id "Connector:Conn_01x04_Male") (at 114.6048 68.9356 0) (unit 1)
     (in_bom yes) (on_board yes) (fields_autoplaced)
-    (property "Reference" "J?" (id 0) (at 115.2398 60.7568 0))
+    (property "Reference" "J1" (id 0) (at 115.2398 60.7568 0))
     (property "Value" "Conn_01x04_Male" (id 1) (at 115.2398 63.2968 0))
     (property "Footprint" "Connector_PinHeader_2.54mm:PinHeader_1x04_P2.54mm_Vertical" (id 2) (at 114.6048 68.9356 0)
